Commit message: added ros2 control interfaces for delta and beckhoff

File: kuka_structure_description/urdf/kuka_structure_robot.xacro (robot description, xacro)
@@ -86,7 +86,7 @@
     </collision>
   </link>
-  <!-- <joint name="${prefix}joint_1" type="prismatic">
+  <joint name="${prefix}joint_1" type="prismatic">
     <origin
-      xyz="2.750 0.215 2.720"
+      xyz="-0.250 0.215 2.720"
       rpy="0 0 0" />
     <parent
@@ -95,5 +95,5 @@
       link="${prefix}link_1" />
     <axis
-      xyz="-1 0 0" />
+      xyz="1 0 0" />
     <limit
       lower="0"
@@ -101,7 +101,7 @@
       effort="${joint_1_eff_limit}"
       velocity="${joint_1_vel_limit}" />
-  </joint> -->
+  </joint>
 <!-- current position -->
-  <joint name="${prefix}joint_1" type="fixed">
+  <!-- <joint name="${prefix}joint_1" type="fixed">
     <origin
       xyz="0.850 0.215 2.720"
@@ -115,8 +115,8 @@
     <limit
       lower="0"
-      upper="3.0"
+      upper="30000000000000.0"
       effort="${joint_1_eff_limit}"
       velocity="${joint_1_vel_limit}" />
-  </joint>
+  </joint> -->
 <!-- end current position -->
 </xacro:macro>

File: kuka_structure_description/urdf/kuka_structure_ros2_control.xacro (robot description, xacro)
@@ -9,5 +9,5 @@
         <xacro:if value="${use_fake_hardware}">
           <plugin>mock_components/GenericSystem</plugin>
-          <param name="fake_sensor_commands">false</param>
+          <param name="mock_sensor_commands">false</param>
           <param name="state_following_offset">0.0</param>
         </xacro:if>
@@ -19,8 +19,19 @@
       </hardware>
       <joint name="${prefix}joint_1">
-        <state_interface name="position"/>
+        <state_interface name="position">
+          <param name="initial_value">0.0</param>
+        </state_interface>
+        <state_interface name="velocity">
+          <param name="initial_value">0.0</param>
+        </state_interface>
+        <state_interface name="effort">
+          <param name="initial_value">0.0</param>
+        </state_interface>
         <state_interface name="status_word"/>
-        <state_interface name="ctrl_word"/>
+        <state_interface name="moo_display"/>
         <command_interface name="position"/>
+        <command_interface name="velocity"/>
+        <command_interface name="ctrl_word"/>
+        <command_interface name="moo"/>
         <ec_module name="${name}">
           <plugin>ethercat_generic_plugins/EcCiA402Drive</plugin>
@@ -28,7 +39,55 @@
           <param name="position">0</param>
           <param name="mode_of_operation">8</param>
-          <param name="slave_config">$(find kuka_structure_description)/config/ethercat_config.yaml</param>
+          <param name="slave_config">$(find kuka_structure_description)/config/delta_ethercat_config.yaml</param>
         </ec_module>
       </joint>
+      <gpio name="digital_inputs">
+        <state_interface name="d_input.0"/>
+        <state_interface name="d_input.1"/>
+        <state_interface name="d_input.2"/>
+        <state_interface name="d_input.3"/>
+        <state_interface name="d_input.4"/>
+        <state_interface name="d_input.5"/>
+        <state_interface name="d_input.6"/>
+        <state_interface name="d_input.7"/>
+        <ec_module name="EL1008">
+          <plugin>ethercat_generic_plugins/GenericEcSlave</plugin>
+          <param name="alias">0</param>
+          <param name="position">2</param>
+          <param name="slave_config">$(find kuka_structure_description)/config/EL1008_ethercat_config.yaml</param>
+        </ec_module>
+      </gpio>
+      <gpio name="digital_outputs1">
+        <command_interface name="d_output.0"/>
+        <command_interface name="d_output.1"/>
+        <command_interface name="d_output.2"/>
+        <command_interface name="d_output.3"/>
+        <command_interface name="d_output.4"/>
+        <command_interface name="d_output.5"/>
+        <command_interface name="d_output.6"/>
+        <command_interface name="d_output.7"/>
+        <ec_module name="EL2008">
+          <plugin>ethercat_generic_plugins/GenericEcSlave</plugin>
+          <param name="alias">0</param>
+          <param name="position">3</param>
+          <param name="slave_config">$(find kuka_structure_description)/config/EL2008_ethercat_config.yaml</param>
+        </ec_module>
+      </gpio>
+      <gpio name="digital_outputs2">
+        <command_interface name="d_output.0"/>
+        <command_interface name="d_output.1"/>
+        <command_interface name="d_output.2"/>
+        <command_interface name="d_output.3"/>
+        <command_interface name="d_output.4"/>
+        <command_interface name="d_output.5"/>
+        <command_interface name="d_output.6"/>
+        <command_interface name="d_output.7"/>
+        <ec_module name="EL2008">
+          <plugin>ethercat_generic_plugins/GenericEcSlave</plugin>
+          <param name="alias">0</param>
+          <param name="position">4</param>
+          <param name="slave_config">$(find kuka_structure_description)/config/EL2008_ethercat_config.yaml</param>
+        </ec_module>
+      </gpio>
     </ros2_control>
   </xacro:macro>

Commit message: Integrated IO beckhoff modules

File: kuka_structure_description/urdf/kuka_structure_robot.xacro (robot description, xacro)
@@ -4,4 +4,6 @@
   <xacro:property name="joint_1_vel_limit" value="1.74533" />    <!--  100°/s -->
   <xacro:property name="joint_1_eff_limit" value="100000" />
+  <xacro:property name="joint_1_lower_position_limit" value="0" />
+  <xacro:property name="joint_1_upper_position_limit" value="2.9" />
   <link name="${prefix}base_link">
     <inertial>
@@ -97,6 +99,6 @@
       xyz="1 0 0" />
     <limit
-      lower="0"
-      upper="3.0"
+      lower="${joint_1_lower_position_limit}"
+      upper="${joint_1_upper_position_limit}"
       effort="${joint_1_eff_limit}"
       velocity="${joint_1_vel_limit}" />

File: kuka_structure_description/urdf/kuka_structure_ros2_control.xacro (robot description, xacro)
@@ -30,4 +30,5 @@
         <state_interface name="status_word"/>
         <state_interface name="moo_display"/>
+        <state_interface name="error_code"/>
         <command_interface name="position"/>
         <command_interface name="velocity"/>
@@ -35,8 +36,8 @@
         <command_interface name="moo"/>
         <ec_module name="${name}">
-          <plugin>ethercat_generic_plugins/EcCiA402Drive</plugin>
+          <plugin>ethercat_generic_plugins/GenericEcSlave</plugin>
           <param name="alias">0</param>
+          <!-- <param name="alias">2</param> -->
           <param name="position">0</param>
-          <param name="mode_of_operation">8</param>
           <param name="slave_config">$(find kuka_structure_description)/config/delta_ethercat_config.yaml</param>
         </ec_module>

Commit message: Linear axis fixed for personal tests

File: kuka_structure_description/urdf/kuka_structure_robot.xacro (robot description, xacro)
@@ -88,5 +88,6 @@
     </collision>
   </link>
-  <joint name="${prefix}joint_1" type="prismatic">
+  <!-- <joint name="${prefix}joint_1" type="prismatic"> -->
+  <joint name="${prefix}joint_1" type="fixed">
     <origin
       xyz="-0.250 0.215 2.720"
