Commit message: working status

File: kuka_structure_description/urdf/kuka_structure_ros2_control.xacro (robot description, xacro)
@@ -28,7 +28,13 @@
           <param name="initial_value">0.0</param>
         </state_interface>
-        <state_interface name="status_word"/>
-        <state_interface name="moo_display"/>
-        <state_interface name="error_code"/>
+        <state_interface name="status_word">
+          <param name="initial_value">0</param>
+        </state_interface>
+        <state_interface name="moo_display">
+          <param name="initial_value">0</param>
+        </state_interface>
+        <state_interface name="error_code">
+          <param name="initial_value">0</param>
+        </state_interface>
         <command_interface name="position"/>
         <command_interface name="velocity"/>
@@ -44,12 +50,28 @@
       </joint>
       <gpio name="digital_inputs">
-        <state_interface name="lubrication_state"/>
-        <state_interface name="limit_switch_homing"/>
-        <state_interface name="limit_switch_end"/>
-        <state_interface name="d_input.3"/>
-        <state_interface name="d_input.4"/>
-        <state_interface name="d_input.5"/>
-        <state_interface name="d_input.6"/>
-        <state_interface name="d_input.7"/>
+        <state_interface name="lubrication_state">
+          <param name="initial_value">0</param>
+        </state_interface>
+        <state_interface name="limit_switch_homing">
+          <param name="initial_value">0</param>
+        </state_interface>
+        <state_interface name="limit_switch_end">
+          <param name="initial_value">0</param>
+        </state_interface>
+        <state_interface name="d_input.3">
+          <param name="initial_value">0</param>
+        </state_interface>
+        <state_interface name="d_input.4">
+          <param name="initial_value">0</param>
+        </state_interface>
+        <state_interface name="d_input.5">
+          <param name="initial_value">0</param>
+        </state_interface>
+        <state_interface name="d_input.6">
+          <param name="initial_value">0</param>
+        </state_interface>
+        <state_interface name="d_input.7">
+          <param name="initial_value">0</param>
+        </state_interface>
         <ec_module name="EL1008">
           <plugin>ethercat_generic_plugins/GenericEcSlave</plugin>
@@ -93,18 +115,46 @@
       <gpio name="analog_inputs">
         <command_interface name="sensor_reset"/>
-        <state_interface name="sensor_channel_0"/>
-        <state_interface name="sensor_channel_1"/>
-        <state_interface name="sensor_channel_2"/>
-        <state_interface name="sensor_channel_3"/>
-        <state_interface name="sensor_channel_4"/>
-        <state_interface name="sensor_channel_5"/>
-        <state_interface name="a_input_6"/>
-        <state_interface name="a_input_7"/>
-        <state_interface name="force_x"/>
-        <state_interface name="force_y"/>
-        <state_interface name="force_z"/>
-        <state_interface name="torque_x"/>
-        <state_interface name="torque_y"/>
-        <state_interface name="torque_z"/>
+        <state_interface name="sensor_channel_0">
+          <param name="initial_value">0.0</param>
+        </state_interface>
+        <state_interface name="sensor_channel_1">
+          <param name="initial_value">0.0</param>
+        </state_interface>
+        <state_interface name="sensor_channel_2">
+          <param name="initial_value">0.0</param>
+        </state_interface>
+        <state_interface name="sensor_channel_3">
+          <param name="initial_value">0.0</param>
+        </state_interface>
+        <state_interface name="sensor_channel_4">
+          <param name="initial_value">0.0</param>
+        </state_interface>
+        <state_interface name="sensor_channel_5">
+          <param name="initial_value">0.0</param>
+        </state_interface>
+        <state_interface name="a_input_6">
+          <param name="initial_value">0.0</param>
+        </state_interface>
+        <state_interface name="a_input_7">
+          <param name="initial_value">0.0</param>
+        </state_interface>
+        <state_interface name="force_x">
+          <param name="initial_value">0.0</param>
+        </state_interface>
+        <state_interface name="force_y">
+          <param name="initial_value">0.0</param>
+        </state_interface>
+        <state_interface name="force_z">
+          <param name="initial_value">0.0</param>
+        </state_interface>
+        <state_interface name="torque_x">
+          <param name="initial_value">0.0</param>
+        </state_interface>
+        <state_interface name="torque_y">
+          <param name="initial_value">0.0</param>
+        </state_interface>
+        <state_interface name="torque_z">
+          <param name="initial_value">0.0</param>
+        </state_interface>
         <ec_module name="EL3008">
           <plugin>ethercat_generic_plugins/EcAtiSensor</plugin>

File: kuka_structure_description/urdf/kuka_structure_rviz.xacro (robot description, xacro)
@@ -2,5 +2,5 @@
 <robot name="kuka_structure" xmlns:xacro="http://www.ros.org/wiki/xacro">
   <xacro:arg name="robot_name" default="kuka_structure"/>
-  <xacro:arg name="prefix" default=""/>
+  <xacro:arg name="prefix" default="structure_"/>
   <xacro:arg name="use_fake_hardware" default="false"/>
   <xacro:property name="prefix" value="'$(arg prefix)'" />

File: kuka_structure_moveit_config/config/kuka_structure.ros2_control.xacro (robot description, xacro)
@@ -8,8 +8,8 @@
                 <plugin>mock_components/GenericSystem</plugin>
             </hardware>
-            <joint name="joint_1">
+            <joint name="structure_joint_1">
                 <command_interface name="position"/>
                 <state_interface name="position">
-                  <param name="initial_value">${initial_positions['joint_1']}</param>
+                  <param name="initial_value">${initial_positions['structure_joint_1']}</param>
                 </state_interface>
                 <state_interface name="velocity"/>
